File: pain5.kicad_pcb (KiCad board)
At the start: 2 copper layers, 110 x 42 mm, 32 parts, among them J1 USB_C_Receptacle_USB2.0, J2 ISP Programming, J3 Reseter, K1 KEYSW, K2 KEYSW, K3 KEYSW, K4 KEYSW, K5 KEYSW, U1 MCU-ATMEGA32U4-MUR(VQFN44), Y1 Crystal_GND24

Commit message: [tweak] rgb update :)
Parts:
- added D10: Inolux_IN-PI554FCH, LED_SMD:LED_Inolux_IN-PI554FCH_PLCC4_5.0x5.0mm_P3.2mm, F.Cu at (184.2, 95.2)
- added D11: Inolux_IN-PI554FCH, LED_SMD:LED_Inolux_IN-PI554FCH_PLCC4_5.0x5.0mm_P3.2mm, F.Cu at (203.3, 95.2)
- added D7: Inolux_IN-PI554FCH, LED_SMD:LED_Inolux_IN-PI554FCH_PLCC4_5.0x5.0mm_P3.2mm, F.Cu at (126.7, 95.2)
- added D8: Inolux_IN-PI554FCH, LED_SMD:LED_Inolux_IN-PI554FCH_PLCC4_5.0x5.0mm_P3.2mm, F.Cu at (145.9, 95.2)
- added D9: Inolux_IN-PI554FCH, LED_SMD:LED_Inolux_IN-PI554FCH_PLCC4_5.0x5.0mm_P3.2mm, F.Cu at (165.0, 95.2)
- added J4: Bootloader, Connector_PinHeader_1.00mm:PinHeader_1x02_P1.00mm_Vertical, F.Cu at (153.6, 78.0)
- added R8: 10K, Resistor_SMD:R_0603_1608Metric, F.Cu at (149.7, 78.0)
- U1: footprint ATMEGA-32U4-MUR:MCU-ATMEGA32U4-MUR_VQFN44 -> ATMEGA-32U4-AU:QFP80P1200X1200X120-44N
- moved C3 22.7 mm to (156.3, 75.0), turned to 90 degrees
- moved C4 18.0 mm to (148.7, 65.7), turned to 270 degrees
- moved C6 15.0 mm to (132.8, 68.6)
- moved C5 11.4 mm to (136.9, 79.6), turned to 180 degrees
- moved J3 9.94 mm to (124.9, 65.3), turned to 270 degrees
- moved R5 6.50 mm to (130.1, 68.5)
- moved C9 6.02 mm to (140.3, 64.0), turned to 180 degrees
- moved J2 5.29 mm to (132.1, 65.3), turned to 270 degrees
- moved R1 4.52 mm to (152.9, 66.4)
- moved R2 4.10 mm to (152.9, 64.9)
- moved C7 3.60 mm to (150.6, 68.6), turned to 90 degrees
- moved Y1 2.61 mm to (126.9, 72.1)
- moved C2 2.61 mm to (127.0, 68.7)
- moved C1 2.61 mm to (126.9, 75.5)
- moved U1 2.26 mm to (141.0, 71.8)
Connections:
- U1 pad 12: Net-(U1-Pad12) -> /RGB_OUT
Routing:
- net VCC: track 98.4 -> 207.7 mm, vias 7 -> 14
- net /RGB_OUT: track 0.00 -> 37.2 mm, vias 0 -> 2
- net GND: track 29.4 -> 12.2 mm
- net Net-(D7-Pad4): track 0.00 -> 15.6 mm
- net Net-(D10-Pad2): track 0.00 -> 15.6 mm
- net Net-(D10-Pad4): track 0.00 -> 15.6 mm
- net Net-(D8-Pad4): track 0.00 -> 15.6 mm
- net Net-(J4-Pad2): track 0.00 -> 8.11 mm
- net /SCK: track 4.59 -> 11.2 mm, vias 0 -> 1
- net /MOSI: track 5.90 -> 10.9 mm, vias 1 -> 0
- net Net-(C9-Pad1): track 6.13 -> 1.91 mm
- net /K1: track 16.4 -> 13.3 mm
- net Net-(J1-PadA7): track 15.8 -> 13.5 mm
- net /RST: track 16.0 -> 14.4 mm, vias 0 -> 2
- net Net-(J1-PadA6): track 16.4 -> 15.1 mm
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Other:
- board text added: "Feb. 2021"
- board text added: "Rev 1.1"
- board text removed: "1"
- board text removed: "6"
- board text removed: "Jan. 2021"
- board text removed: "Prototype"
- board text removed: "Rev. P1"
