File: pain5.sch (KiCad schematic (older format))
At the start: 28 parts, among them J1 USB_C_Receptacle_USB2.0, J2 ISP Programming, J3 Reseter, K1 KEYSW, K2 KEYSW, K3 KEYSW, K4 KEYSW, K5 KEYSW, U1 MCU-ATMEGA32U4-MUR(VQFN44), Y1 Crystal_GND24

Commit message: [tweak] i don't wanna write it all
Parts:
- K1, K2, K3, K4, K5: footprint Switch_Keyboard_Cherry_MX:SW_Cherry_MX_PCB_1.00u -> (none)
- U1: footprint k-5:QFN44G-0.5-7X7MM -> QFN44G-0.5-7X7MM; LCSC C45874 -> (none); MPN (none) -> ATMEGA32U4-MUR
Changed lines of the file:
@@
 Wire Wire Line
 	5100 2150 5100 2250
-$Comp
-L MCU-ATMEGA32U4-MUR_VQFN44_:MCU-ATMEGA32U4-MUR(VQFN44) U1
-U 1 1 5FC48137
-P 6400 3450
-F 0 "U1" H 6350 5117 50  0000 C CNN
-F 1 "MCU-ATMEGA32U4-MUR(VQFN44)" H 6350 5026 50  0000 C CNN
-F 2 "k-5:QFN44G-0.5-7X7MM" H 6400 3450 50  0001 L BNN
-F 3 "" H 6400 3450 50  0001 L BNN
-F 4 "C45874" H 6400 3450 50  0001 L BNN "LCSC"
-	1    6400 3450
-	1    0    0    -1
-$EndComp
 Wire Wire Line
 	5000 2350 5100 2350
@@
 F 4 "C170140" H 3750 1000 50  0001 C CNN "LCSC"
 	1    3750 1000
-	1    0    0    -1
-$EndComp
-$Comp
-L keyboard_parts:KEYSW K1
-U 1 1 5FCFEDF5
-P 10250 2500
-F 0 "K1" H 10250 2733 60  0000 C CNN
-F 1 "KEYSW" H 10250 2400 60  0001 C CNN
-F 2 "Switch_Keyboard_Cherry_MX:SW_Cherry_MX_PCB_1.00u" H 10250 2500 60  0001 C CNN
-F 3 "" H 10250 2500 60  0000 C CNN
-	1    10250 2500
-	1    0    0    -1
-$EndComp
-$Comp
-L keyboard_parts:KEYSW K2
-U 1 1 5FD03101
-P 10250 2900
-F 0 "K2" H 10250 3133 60  0000 C CNN
-F 1 "KEYSW" H 10250 2800 60  0001 C CNN
-F 2 "Switch_Keyboard_Cherry_MX:SW_Cherry_MX_PCB_1.00u" H 10250 2900 60  0001 C CNN
-F 3 "" H 10250 2900 60  0000 C CNN
-	1    10250 2900
-	1    0    0    -1
-$EndComp
-$Comp
-L keyboard_parts:KEYSW K3
-U 1 1 5FD03E85
-P 10250 3350
-F 0 "K3" H 10250 3583 60  0000 C CNN
-F 1 "KEYSW" H 10250 3250 60  0001 C CNN
-F 2 "Switch_Keyboard_Cherry_MX:SW_Cherry_MX_PCB_1.00u" H 10250 3350 60  0001 C CNN
-F 3 "" H 10250 3350 60  0000 C CNN
-	1    10250 3350
-	1    0    0    -1
-$EndComp
-$Comp
-L keyboard_parts:KEYSW K4
-U 1 1 5FD04C6C
-P 10250 3800
-F 0 "K4" H 10250 4033 60  0000 C CNN
-F 1 "KEYSW" H 10250 3700 60  0001 C CNN
-F 2 "Switch_Keyboard_Cherry_MX:SW_Cherry_MX_PCB_1.00u" H 10250 3800 60  0001 C CNN
-F 3 "" H 10250 3800 60  0000 C CNN
-	1    10250 3800
-	1    0    0    -1
-$EndComp
-$Comp
-L keyboard_parts:KEYSW K5
-U 1 1 5FD06371
-P 10250 4250
-F 0 "K5" H 10250 4483 60  0000 C CNN
-F 1 "KEYSW" H 10250 4150 60  0001 C CNN
-F 2 "Switch_Keyboard_Cherry_MX:SW_Cherry_MX_PCB_1.00u" H 10250 4250 60  0001 C CNN
-F 3 "" H 10250 4250 60  0000 C CNN
-	1    10250 4250
 	1    0    0    -1
 $EndComp
@@
 Text Label 10550 2150 1    50   ~ 0
 KVCC
-Wire Wire Line
-	10550 2150 10550 2500
-Connection ~ 10550 2500
-Wire Wire Line
-	10550 2500 10550 2900
-Connection ~ 10550 2900
-Wire Wire Line
-	10550 2900 10550 3350
-Connection ~ 10550 3350
-Wire Wire Line
-	10550 3350 10550 3800
-Connection ~ 10550 3800
-Wire Wire Line
-	10550 3800 10550 4250
 Wire Wire Line
 	9500 2500 9350 2500
@@
 Wire Wire Line
 	2950 3250 3050 3250
+$Comp
+L MCU-ATMEGA32U4-MUR_VQFN44_:MCU-ATMEGA32U4-MUR(VQFN44) U1
+U 1 1 5FE16671
+P 6400 3450
+F 0 "U1" H 6350 5117 50  0000 C CNN
+F 1 "MCU-ATMEGA32U4-MUR(VQFN44)" H 6350 5026 50  0000 C CNN
+F 2 "QFN44G-0.5-7X7MM" H 6400 3450 50  0001 L BNN
+F 3 "" H 6400 3450 50  0001 L BNN
+F 4 "ATMEGA32U4-MUR" H 6400 3450 50  0001 L BNN "MPN"
+	1    6400 3450
+	1    0    0    -1
+$EndComp
+Wire Wire Line
+	10550 2150 10550 2500
+$Comp
+L keyboard_parts:KEYSW K1
+U 1 1 5FE1C4F5
+P 10250 2500
+F 0 "K1" H 10250 2733 60  0000 C CNN
+F 1 "KEYSW" H 10250 2400 60  0001 C CNN
+F 2 "" H 10250 2500 60  0000 C CNN
+F 3 "" H 10250 2500 60  0000 C CNN
+	1    10250 2500
+	1    0    0    -1
+$EndComp
+Connection ~ 10550 2500
+Wire Wire Line
+	10550 2500 10550 2900
+$Comp
+L keyboard_parts:KEYSW K2
+U 1 1 5FE1D3C3
+P 10250 2900
+F 0 "K2" H 10250 3133 60  0000 C CNN
+F 1 "KEYSW" H 10250 2800 60  0001 C CNN
+F 2 "" H 10250 2900 60  0000 C CNN
+F 3 "" H 10250 2900 60  0000 C CNN
+	1    10250 2900
+	1    0    0    -1
+$EndComp
+Connection ~ 10550 2900
+Wire Wire Line
+	10550 2900 10550 3350
+$Comp
+L keyboard_parts:KEYSW K3
+U 1 1 5FE1DDBE
+P 10250 3350
+F 0 "K3" H 10250 3583 60  0000 C CNN
+F 1 "KEYSW" H 10250 3250 60  0001 C CNN
+F 2 "" H 10250 3350 60  0000 C CNN
+F 3 "" H 10250 3350 60  0000 C CNN
+	1    10250 3350
+	1    0    0    -1
+$EndComp
+Connection ~ 10550 3350
+Wire Wire Line
+	10550 3350 10550 3800
+$Comp
+L keyboard_parts:KEYSW K4
+U 1 1 5FE1EEB4
+P 10250 3800
+F 0 "K4" H 10250 4033 60  0000 C CNN
+F 1 "KEYSW" H 10250 3700 60  0001 C CNN
+F 2 "" H 10250 3800 60  0000 C CNN
+F 3 "" H 10250 3800 60  0000 C CNN
+	1    10250 3800
+	1    0    0    -1
+$EndComp
+Connection ~ 10550 3800
+Wire Wire Line
+	10550 3800 10550 4250
+$Comp
+L keyboard_parts:KEYSW K5
+U 1 1 5FE1FAEC
+P 10250 4250
+F 0 "K5" H 10250 4483 60  0000 C CNN
+F 1 "KEYSW" H 10250 4150 60  0001 C CNN
+F 2 "" H 10250 4250 60  0000 C CNN
+F 3 "" H 10250 4250 60  0000 C CNN
+	1    10250 4250
+	1    0    0    -1
+$EndComp
 $EndSCHEMATC

Commit message: [upload] added a lot more
Parts:
- added D6: POWER_LED, LED_SMD:LED_0603_1608Metric, symbol Device:LED
- added R5: 10K, Resistor_SMD:R_0603_1608Metric, symbol Device:R
- added R6: 1K, Resistor_SMD:R_0603_1608Metric, symbol Device:R
- added R7: 2K, Resistor_SMD:R_0603_1608Metric, symbol Device:R
- J2: footprint Connector_PinHeader_1.00mm:PinHeader_2x03_P1.00mm_Vertical -> Connector_PinHeader_1.00mm:PinHeader_1x06_P1.00mm_Vertical
- K1, K2, K3, K4, K5: footprint (none) -> Switch_Keyboard_Cherry_MX:SW_Cherry_MX_PCB_1.00u
- U1: footprint QFN44G-0.5-7X7MM -> ATMEGA-32U4-MUR:MCU-ATMEGA32U4-MUR_VQFN44
- Y1: footprint Crystals:Crystal_SMD_3225-4Pin_3.2x2.5mm -> Crystal:Crystal_SMD_3225-4Pin_3.2x2.5mm
Connections:
- net GND: now also D6.1 (K), R7.2
- net K2: now also U1.26 (PD6(T1/ADC9/~OC4D)); no longer U1.19 (PD1(SDA/INT1))
- net K3: now also U1.27 (PD7(T0/OC4D/ADC10)); no longer U1.20 (PD2(RXD1/INT2))
- net K4: now also U1.28 (PB4(PCINT4/ADC11)); no longer U1.21 (PD3(TXD1/INT3))
- net K5: now also U1.30 (PB6(PCINT6/OC1B/OC4B/ADC13)); no longer U1.25 (PD4(ICP1/ADC8))
- net KVCC: now also U1.25 (PD4(ICP1/ADC8)); no longer U1.41 (PF0(ADC0))
- net RST: now also R5.2
- net VCC: now also R5.1, R6.1
- new net: D6.2 (A), R6.2, R7.1
- no-connect marks 20 -> 4
Other:
- moved on the sheet: C1, C2, D1, D2, D3, D4, D5, K1, K2, K3, K4, K5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

Commit message: [tweak] rgb update :)
Parts:
- added D10, D11, D7, D8, D9: Inolux_IN-PI554FCH, LED_SMD:LED_Inolux_IN-PI554FCH_PLCC4_5.0x5.0mm_P3.2mm, symbol LED:Inolux_IN-PI554FCH
- added J4: Bootloader, Connector_PinHeader_1.00mm:PinHeader_1x02_P1.00mm_Vertical, symbol Connector_Generic:Conn_02x01
- added R8: 10K, Resistor_SMD:R_0603_1608Metric, symbol Device:R
- D6: LCSC (none) -> C72043
- R5: LCSC (none) -> C25804
- R6: LCSC (none) -> C21190
- R7: LCSC (none) -> C22975
- U1: footprint ATMEGA-32U4-MUR:MCU-ATMEGA32U4-MUR_VQFN44 -> ATMEGA-32U4-AU:QFP80P1200X1200X120-44N; LCSC (none) -> C45874
Connections:
- net GND: now also D10.1 (VSS), D11.1 (VSS), D7.1 (VSS), D8.1 (VSS), D9.1 (VSS), J4.1 (Pin_1)
- net VCC: now also D10.3 (VDD), D11.3 (VDD), D7.3 (VDD), D8.3 (VDD), D9.3 (VDD), R8.1
- net RGB_OUT: now reaches U1.12 (PB7(PCINT7/OC0A/OC1C/~RTS))
- net RGB_OUT: now also D7.2 (DIN)
- net at U1.33 (PE2(~HWB)): now also J4.2 (Pin_2), R8.2
- new net: D7.4 (DO), D8.2 (DIN)
- new net: D8.4 (DO), D9.2 (DIN)
- new net: D10.2 (DIN), D9.4 (DO)
- new net: D10.4 (DO), D11.2 (DIN)
Other:
- moved on the sheet: C3, D1, D2, D3, D4, D5, J1, J2, K1, K2, K3, K4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
